File: Schema/SchemaPCB1.sch (EAGLE design)
At the start: 22 parts, among them J1 CON-HIROSE-COAXIAL-U.FL, J2 Programmer, U1 RN2483, U2 TPS22860DBVR, U3 ESP32-WROOM-32E_M113EH3200PH3Q, U4 SOT-89-5, U5 SI7217-B-01-IVR

Commit message: Board begonnen
Parts:
- U3: value ESP32-WROOM-32E_M113EH3200PH3Q -> ESP32
Connections:
- removed net RXD: U1.UART_TX
- removed net TXD: U1.UART_RX
- new net RXD2: U1.UART_TX, U3.IO16
- new net TXD2: U1.UART_RX, U3.IO17
- net +3V3: now also J2.4; no longer J2.5
- net GND: now also J2.5; no longer J2.4
- net I2C_SCL: now also J3.8
- net I2C_SDA: no longer J3.8
- net RN2483_ENABLE: now also U3.IO19; no longer U3.IO16
- net RN2483_RESET: now also U3.IO18; no longer U3.IO17
Changed lines of the file:
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@@
 <drawing>
 <settings>
-<setting alwaysvectorfont="yes"/>
+<setting alwaysvectorfont="no"/>
 <setting keepoldvectorfont="yes"/>
 <setting verticaltext="up"/>
@@
 </classes>
 <parts>
-<part name="U3" library="--CoolTeamLib" deviceset="ESP32-WROOM-32E_M113EH3200PH3Q" device=""/>
+<part name="U3" library="--CoolTeamLib" deviceset="ESP32-WROOM-32E_M113EH3200PH3Q" device="" value="ESP32"/>
 <part name="GND1" library="supply1" library_urn="urn:adsk.eagle:library:371" deviceset="GND" device=""/>
 <part name="GND2" library="supply1" library_urn="urn:adsk.eagle:library:371" deviceset="GND" device=""/>
@@
 <attribute name="NAME" x="48.26" y="61.468" size="1.778" layer="95" font="vector"/>
 </instance>
-<instance part="GND6" gate="1" x="96.52" y="50.8" smashed="yes">
-<attribute name="VALUE" x="93.98" y="48.26" size="1.778" layer="96"/>
+<instance part="GND6" gate="1" x="63.5" y="58.42" smashed="yes">
+<attribute name="VALUE" x="60.96" y="55.88" size="1.778" layer="96"/>
 </instance>
 <instance part="+3V6" gate="G$1" x="73.66" y="66.04" smashed="yes">
@@
 </segment>
 <segment>
-<pinref part="J2" gate="G$1" pin="4"/>
-<pinref part="GND6" gate="1" pin="GND"/>
-<wire x1="58.42" y1="55.88" x2="96.52" y2="55.88" width="0.1524" layer="91"/>
-<wire x1="96.52" y1="55.88" x2="96.52" y2="53.34" width="0.1524" layer="91"/>
-</segment>
-<segment>
 <pinref part="J3" gate="G$1" pin="9"/>
 <wire x1="213.36" y1="71.12" x2="243.84" y2="71.12" width="0.1524" layer="91"/>
@@
 <wire x1="139.7" y1="177.8" x2="139.7" y2="175.26" width="0.1524" layer="91"/>
 <junction x="139.7" y="177.8"/>
+</segment>
+<segment>
+<pinref part="J2" gate="G$1" pin="5"/>
+<wire x1="58.42" y1="58.42" x2="58.42" y2="60.96" width="0.1524" layer="91"/>
+<pinref part="GND6" gate="1" pin="GND"/>
+<wire x1="58.42" y1="60.96" x2="63.5" y2="60.96" width="0.1524" layer="91"/>
 </segment>
 </net>
@@
 </segment>
 <segment>
-<pinref part="J2" gate="G$1" pin="5"/>
-<wire x1="58.42" y1="58.42" x2="73.66" y2="58.42" width="0.1524" layer="91"/>
 <pinref part="+3V6" gate="G$1" pin="+3V3"/>
-<wire x1="73.66" y1="58.42" x2="73.66" y2="63.5" width="0.1524" layer="91"/>
+<wire x1="73.66" y1="55.88" x2="73.66" y2="63.5" width="0.1524" layer="91"/>
+<pinref part="J2" gate="G$1" pin="4"/>
+<wire x1="58.42" y1="55.88" x2="73.66" y2="55.88" width="0.1524" layer="91"/>
 </segment>
 <segment>
@@
 </segment>
 </net>
-<net name="RN2483_ENABLE" class="0">
-<segment>
-<pinref part="U3" gate="G$1" pin="IO16"/>
-<wire x1="165.1" y1="127" x2="175.26" y2="127" width="0.1524" layer="91"/>
-<label x="175.26" y="127" size="1.778" layer="95"/>
-</segment>
-</net>
-<net name="RN2483_RESET" class="0">
-<segment>
-<pinref part="U3" gate="G$1" pin="IO17"/>
-<wire x1="165.1" y1="124.46" x2="175.26" y2="124.46" width="0.1524" layer="91"/>
-<label x="175.26" y="124.46" size="1.778" layer="95"/>
-</segment>
-</net>
 <net name="HALL_EN" class="0">
 <segment>
@@
 <junction x="213.36" y="104.14"/>
 </segment>
+<segment>
+<pinref part="J3" gate="G$1" pin="8"/>
+<wire x1="213.36" y1="68.58" x2="223.52" y2="68.58" width="0.1524" layer="91"/>
+<label x="223.52" y="68.58" size="1.778" layer="95"/>
+</segment>
 </net>
 <net name="I2C_SDA" class="0">
@@
 <wire x1="223.52" y1="114.3" x2="223.52" y2="111.76" width="0.1524" layer="91"/>
 <junction x="223.52" y="111.76"/>
-</segment>
-<segment>
-<pinref part="J3" gate="G$1" pin="8"/>
-<wire x1="213.36" y1="68.58" x2="223.52" y2="68.58" width="0.1524" layer="91"/>
-<label x="223.52" y="68.58" size="1.778" layer="95"/>
 </segment>
 <segment>
@@
 <pinref part="J3" gate="G$1" pin="2"/>
 <wire x1="213.36" y1="53.34" x2="223.52" y2="53.34" width="0.1524" layer="91"/>
+</segment>
+</net>
+<net name="RXD2" class="0">
+<segment>
+<pinref part="U3" gate="G$1" pin="IO16"/>
+<wire x1="165.1" y1="127" x2="175.26" y2="127" width="0.1524" layer="91"/>
+<label x="175.26" y="127" size="1.778" layer="95"/>
+</segment>
+</net>
+<net name="TXD2" class="0">
+<segment>
+<pinref part="U3" gate="G$1" pin="IO17"/>
+<wire x1="165.1" y1="124.46" x2="175.26" y2="124.46" width="0.1524" layer="91"/>
+<label x="175.26" y="124.46" size="1.778" layer="95"/>
+</segment>
+</net>
+<net name="RN2483_RESET" class="0">
+<segment>
+<pinref part="U3" gate="G$1" pin="IO18"/>
+<wire x1="165.1" y1="119.38" x2="175.26" y2="119.38" width="0.1524" layer="91"/>
+<label x="175.26" y="119.38" size="1.778" layer="95"/>
+</segment>
+</net>
+<net name="RN2483_ENABLE" class="0">
+<segment>
+<pinref part="U3" gate="G$1" pin="IO19"/>
+<wire x1="165.1" y1="116.84" x2="175.26" y2="116.84" width="0.1524" layer="91"/>
+<label x="175.26" y="116.84" size="1.778" layer="95"/>
 </segment>
 </net>
@@
 </segment>
 </net>
-<net name="RXD" class="0">
+<net name="RXD2" class="0">
 <segment>
 <pinref part="U1" gate="G$1" pin="UART_TX"/>
@@
 </segment>
 </net>
-<net name="TXD" class="0">
+<net name="TXD2" class="0">
 <segment>
 <pinref part="U1" gate="G$1" pin="UART_RX"/>

Commit message: gps toegevoegd
Parts:
- added C10: 0.1uF, ngspice-simulation:C
- added C11: 1uF, ngspice-simulation:C
- added R4, R5: 10k, ngspice-simulation:R
- added T1: (no value), zetex:PMOSSOT23
- added U?1: GPS, gps:GPS
Connections:
- new net *GPS_ENABLE: T1.G, U3.NC_7
- new net N$5: R4.1, U?1.WAKE-UP
- new net N$6: R5.1, U?1.NRESET
- new net N$8: C10.1, C11.1, R5.2, T1.S, U?1.VCC
- net +3V3: now also T1.D
- net GND: now also C10.2, C11.2, R4.2, U?1.GND
- net I2C_SCL: now also U?1.I2C_SCL
- net I2C_SDA: now also U?1.I2C_SDA
Changed lines of the file:
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@@
 <part name="GND8" library="supply1" library_urn="urn:adsk.eagle:library:371" deviceset="GND" device=""/>
 <part name="GND9" library="supply1" library_urn="urn:adsk.eagle:library:371" deviceset="GND" device=""/>
+<part name="GND10" library="supply1" library_urn="urn:adsk.eagle:library:371" deviceset="GND" device=""/>
+<part name="+3V8" library="supply1" library_urn="urn:adsk.eagle:library:371" deviceset="+3V3" device=""/>
+<part name="T1" library="zetex" library_urn="urn:adsk.eagle:library:418" deviceset="PMOSSOT23" device="" package3d_urn="urn:adsk.eagle:package:30981/1"/>
+<part name="R5" library="ngspice-simulation" library_urn="urn:adsk.eagle:library:527439" deviceset="R" device="" value="10k"/>
+<part name="C10" library="ngspice-simulation" library_urn="urn:adsk.eagle:library:527439" deviceset="C" device="" value="0.1uF"/>
+<part name="C11" library="ngspice-simulation" library_urn="urn:adsk.eagle:library:527439" deviceset="C" device="" value="1uF"/>
+<part name="GND16" library="supply1" library_urn="urn:adsk.eagle:library:371" deviceset="GND" device=""/>
+<part name="R4" library="ngspice-simulation" library_urn="urn:adsk.eagle:library:527439" deviceset="R" device="" value="10k"/>
+<part name="GND15" library="supply1" library_urn="urn:adsk.eagle:library:371" deviceset="GND" device=""/>
+<part name="U?1" library="gps" deviceset="GPS" device=""/>
 </parts>
 <sheets>
@@
 </segment>
 </net>
+<net name="*GPS_ENABLE" class="0">
+<segment>
+<pinref part="U3" gate="G$1" pin="NC_7"/>
+<wire x1="165.1" y1="114.3" x2="175.26" y2="114.3" width="0.1524" layer="91"/>
+<label x="175.26" y="114.3" size="1.778" layer="95"/>
+</segment>
+</net>
 </nets>
 </sheet>
@@
 <attribute name="DRAWING_NAME" x="190.5" y="19.05" size="2.54" layer="94"/>
 </instance>
+<instance part="GND10" gate="1" x="144.78" y="116.84" smashed="yes" rot="R90"/>
+<instance part="+3V8" gate="G$1" x="172.72" y="154.94" smashed="yes">
+<attribute name="VALUE" x="170.18" y="149.86" size="1.778" layer="96" rot="R90"/>
+</instance>
+<instance part="T1" gate="A" x="172.72" y="144.78" smashed="yes">
+<attribute name="VALUE" x="175.26" y="144.78" size="1.778" layer="96"/>
+<attribute name="NAME" x="175.26" y="147.32" size="1.778" layer="95"/>
+</instance>
+<instance part="R5" gate="G$1" x="142.24" y="111.76" smashed="yes">
+<attribute name="NAME" x="139.7" y="114.3" size="1.778" layer="95"/>
+<attribute name="VALUE" x="139.7" y="107.95" size="1.778" layer="96"/>
+</instance>
+<instance part="C10" gate="G$1" x="162.56" y="129.54" smashed="yes">
+<attribute name="NAME" x="165.1" y="132.08" size="1.778" layer="95"/>
+<attribute name="VALUE" x="165.1" y="129.54" size="1.778" layer="96"/>
+</instance>
+<instance part="C11" gate="G$1" x="170.18" y="129.54" smashed="yes">
+<attribute name="NAME" x="172.72" y="132.08" size="1.778" layer="95"/>
+<attribute name="VALUE" x="172.72" y="129.54" size="1.778" layer="96"/>
+</instance>
+<instance part="GND16" gate="1" x="167.64" y="119.38" smashed="yes">
+<attribute name="VALUE" x="165.1" y="116.84" size="1.778" layer="96"/>
+</instance>
+<instance part="R4" gate="G$1" x="142.24" y="121.92" smashed="yes">
+<attribute name="NAME" x="139.7" y="124.46" size="1.778" layer="95"/>
+<attribute name="VALUE" x="139.7" y="118.11" size="1.778" layer="96"/>
+</instance>
+<instance part="GND15" gate="1" x="149.86" y="121.92" smashed="yes" rot="R90">
+<attribute name="VALUE" x="152.4" y="119.38" size="1.778" layer="96" rot="R90"/>
+</instance>
+<instance part="U?1" gate="G$1" x="269.24" y="114.3" smashed="yes"/>
 </instances>
 <busses>
 </busses>
 <nets>
+<net name="I2C_SDA" class="0">
+<segment>
+<wire x1="93.98" y1="132.08" x2="83.82" y2="132.08" width="0.1524" layer="91"/>
+<label x="83.82" y="132.08" size="1.778" layer="95" rot="R180"/>
+<pinref part="U?1" gate="G$1" pin="I2C_SDA"/>
+</segment>
+</net>
+<net name="I2C_SCL" class="0">
+<segment>
+<wire x1="93.98" y1="127" x2="83.82" y2="127" width="0.1524" layer="91"/>
+<label x="83.82" y="127" size="1.778" layer="95" rot="R180"/>
+<pinref part="U?1" gate="G$1" pin="I2C_SCL"/>
+</segment>
+</net>
+<net name="GND" class="0">
+<segment>
+<wire x1="132.08" y1="116.84" x2="142.24" y2="116.84" width="0.1524" layer="91"/>
+<pinref part="GND10" gate="1" pin="GND"/>
+<pinref part="U?1" gate="G$1" pin="GND"/>
+</segment>
+<segment>
+<wire x1="170.18" y1="124.46" x2="170.18" y2="121.92" width="0.1524" layer="91"/>
+<pinref part="C11" gate="G$1" pin="2"/>
+<wire x1="170.18" y1="121.92" x2="167.64" y2="121.92" width="0.1524" layer="91"/>
+<pinref part="GND16" gate="1" pin="GND"/>
+<wire x1="162.56" y1="121.92" x2="167.64" y2="121.92" width="0.1524" layer="91"/>
+<wire x1="162.56" y1="124.46" x2="162.56" y2="121.92" width="0.1524" layer="91"/>
+<pinref part="C10" gate="G$1" pin="2"/>
+<junction x="167.64" y="121.92"/>
+</segment>
+<segment>
+<pinref part="R4" gate="G$1" pin="2"/>
+<pinref part="GND15" gate="1" pin="GND"/>
+</segment>
+</net>
+<net name="+3V3" class="0">
+<segment>
+<pinref part="+3V8" gate="G$1" pin="+3V3"/>
+<pinref part="T1" gate="A" pin="D"/>
+<wire x1="172.72" y1="152.4" x2="172.72" y2="149.86" width="0.1524" layer="91"/>
+</segment>
+</net>
+<net name="*GPS_ENABLE" class="0">
+<segment>
+<pinref part="T1" gate="A" pin="G"/>
+<wire x1="167.64" y1="142.24" x2="160.02" y2="142.24" width="0.1524" layer="91"/>
+<label x="160.02" y="142.24" size="1.778" layer="95" rot="R180"/>
+</segment>
+</net>
+<net name="N$6" class="0">
+<segment>
+<wire x1="132.08" y1="111.76" x2="137.16" y2="111.76" width="0.1524" layer="91"/>
+<pinref part="R5" gate="G$1" pin="1"/>
+<pinref part="U?1" gate="G$1" pin="NRESET"/>
+</segment>
+</net>
+<net name="N$8" class="0">
+<segment>
+<wire x1="152.4" y1="132.08" x2="152.4" y2="111.76" width="0.1524" layer="91"/>
+<pinref part="R5" gate="G$1" pin="2"/>
+<wire x1="147.32" y1="111.76" x2="152.4" y2="111.76" width="0.1524" layer="91"/>
+<wire x1="132.08" y1="132.08" x2="152.4" y2="132.08" width="0.1524" layer="91"/>
+<pinref part="T1" gate="A" pin="S"/>
+<wire x1="172.72" y1="139.7" x2="172.72" y2="132.08" width="0.1524" layer="91"/>
+<wire x1="172.72" y1="132.08" x2="170.18" y2="132.08" width="0.1524" layer="91"/>
+<junction x="152.4" y="132.08"/>
+<pinref part="C10" gate="G$1" pin="1"/>
+<wire x1="170.18" y1="132.08" x2="162.56" y2="132.08" width="0.1524" layer="91"/>
+<wire x1="162.56" y1="132.08" x2="152.4" y2="132.08" width="0.1524" layer="91"/>
+<junction x="162.56" y="132.08"/>
+<pinref part="C11" gate="G$1" pin="1"/>
+<junction x="170.18" y="132.08"/>
+<pinref part="U?1" gate="G$1" pin="VCC"/>
+</segment>
+</net>
+<net name="N$5" class="0">
+<segment>
+<pinref part="R4" gate="G$1" pin="1"/>
+<wire x1="132.08" y1="121.92" x2="137.16" y2="121.92" width="0.1524" layer="91"/>
+<pinref part="U?1" gate="G$1" pin="WAKE-UP"/>
+</segment>
+</net>
 </nets>
 </sheet>
