File: Schema/SchemaPCB1.sch (EAGLE design)
At the start: 31 parts, among them J1 CON-HIROSE-COAXIAL-U.FL, J2 Programmer, J4 39700-0205, J5 39700-0002, U1 RN2483, U2 TPS22860DBVR, U3 ESP32, U4 SOT-89-5, U5 SI7217-B-01-IVR, U6 TPS22860DBVR

Commit message: aangepast om te gebruiken met gps breakout board
Parts:
- removed C10, C12: (no value), rcl:C-EUC0805
- removed L1: BLM15HB121SN1, inductors:BLM15HB121SN1
- removed R6, R7: (no value), rcl:R-EU_R0805
- removed U?1: GPS, gps:GPS
- added R2, R3: (no value), rcl:R-EU_R0805
- added U7: ADAFRUIT_MINIGPS, gps:ADAFRUIT_MINIGPS
Connections:
- removed net N$6: C10.1, C12.1, L1.1, U?1.NRESET, U?1.VCC
- removed net N$7: C11.1, L1.2, U6.VOUT
- new net GPS_EN: C11.1, U6.VOUT, U7.*RST, U7.VIN
- net +3V3: now also R2.2, R3.2; no longer R6.2, R7.2
- net GND: now also U7.GND; no longer C10.2, C12.2, U?1.GND, U?1.WAKE-UP
- net I2C_SCL: now also R2.1, U7.SCL; no longer R6.1, U?1.I2C_SCL
- net I2C_SDA: now also R3.1, U7.SDA; no longer R7.1, U?1.I2C_SDA

Commit message: gerber files geexporteerd
Parts:
- C11: value (none) -> 100nF
- C13: value (none) -> 1uF
- R2, R3: value (none) -> 10k
Changed lines of the file:
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@@
 <setting verticaltext="up"/>
 </settings>
-<grid distance="1" unitdist="mm" unit="mm" style="lines" multiple="1" display="no" altdistance="0.1" altunitdist="mm" altunit="mm"/>
+<grid distance="0.1" unitdist="inch" unit="inch" style="lines" multiple="1" display="no" altdistance="0.01" altunitdist="inch" altunit="inch"/>
 <layers>
 <layer number="1" name="Top" color="4" fill="1" visible="no" active="no"/>
@@
 <part name="U6" library="--CoolTeamLib" deviceset="TPS22860DBVR" device=""/>
 <part name="GND17" library="supply1" library_urn="urn:adsk.eagle:library:371" deviceset="GND" device=""/>
-<part name="C11" library="rcl" library_urn="urn:adsk.eagle:library:334" deviceset="C-EU" device="C0805" package3d_urn="urn:adsk.eagle:package:23617/2"/>
-<part name="C13" library="rcl" library_urn="urn:adsk.eagle:library:334" deviceset="C-EU" device="C0805" package3d_urn="urn:adsk.eagle:package:23617/2"/>
+<part name="C11" library="rcl" library_urn="urn:adsk.eagle:library:334" deviceset="C-EU" device="C0805" package3d_urn="urn:adsk.eagle:package:23617/2" value="100nF"/>
+<part name="C13" library="rcl" library_urn="urn:adsk.eagle:library:334" deviceset="C-EU" device="C0805" package3d_urn="urn:adsk.eagle:package:23617/2" value="1uF"/>
 <part name="GND18" library="supply1" library_urn="urn:adsk.eagle:library:371" deviceset="GND" device=""/>
 <part name="+3V2" library="supply1" library_urn="urn:adsk.eagle:library:371" deviceset="+3V3" device=""/>
@@
 <part name="J5" library="--CoolTeamLib" deviceset="39700-0002" device=""/>
 <part name="GND22" library="supply1" library_urn="urn:adsk.eagle:library:371" deviceset="GND" device=""/>
-<part name="R2" library="rcl" library_urn="urn:adsk.eagle:library:334" deviceset="R-EU_" device="R0805" package3d_urn="urn:adsk.eagle:package:23553/2"/>
-<part name="R3" library="rcl" library_urn="urn:adsk.eagle:library:334" deviceset="R-EU_" device="R0805" package3d_urn="urn:adsk.eagle:package:23553/2"/>
+<part name="R2" library="rcl" library_urn="urn:adsk.eagle:library:334" deviceset="R-EU_" device="R0805" package3d_urn="urn:adsk.eagle:package:23553/2" value="10k"/>
+<part name="R3" library="rcl" library_urn="urn:adsk.eagle:library:334" deviceset="R-EU_" device="R0805" package3d_urn="urn:adsk.eagle:package:23553/2" value="10k"/>
 <part name="+3V12" library="supply1" library_urn="urn:adsk.eagle:library:371" deviceset="+3V3" device=""/>
 <part name="+3V13" library="supply1" library_urn="urn:adsk.eagle:library:371" deviceset="+3V3" device=""/>
